Commit message: modified:   plugins/moveit_task_constructor 	new file:   plugins/warehouse_ros_mongo 	modified:   ur5/mycobot_description/config/initial_positions.yaml 	modified:   ur5/mycobot_description/urdf/ur.ros2_control.xacro 	modified:   ur5/mycobot_description/urdf/ur5_robotiq85_gripper.urdf.xacro 	new file:   ur5/mycobot_gripper_description/meshes/campus02_coupler.dae 	modified:   ur5/mycobot_gripper_description/meshes/campus02_coupler.stl 	modified:   ur5/mycobot_moveit/config/controllers.yaml 	modified:   ur5/mycobot_moveit/config/ros2_controllers.yaml 	modified:   ur5/mycobot_moveit/srdf/ur_gripper_macro.srdf.xacro 	modified:   ur5/mycobot_mtc/launch/run.launch.py 	modified:   ur5/mycobot_mtc/package.xml 	modified:   ur5/mycobot_mtc/rviz/mtc_rviz.rviz 	modified:   ur5/mycobot_mtc/src/mtc_node.cpp

File: ur5/mycobot_description/urdf/ur.ros2_control.xacro (robot description, xacro)
@@ -191,4 +191,16 @@
       </joint>
       <joint name="${prefix}robotiq_85_right_finger_joint">
+        <param name="mimic">robotiq_85_left_knuckle_joint</param>
+        <param name="multiplier">-1.0</param>
+        <state_interface name="position"/>
+        <state_interface name="velocity"/>
+      </joint>
+      <joint name="${prefix}robotiq_85_left_finger_tip_joint">
+        <param name="mimic">robotiq_85_left_knuckle_joint</param>
+        <param name="multiplier">-1.0</param>
+        <state_interface name="position"/>
+        <state_interface name="velocity"/>
+      </joint>
+      <joint name="${prefix}robotiq_85_right_finger_tip_joint">
         <param name="mimic">robotiq_85_left_knuckle_joint</param>
         <param name="multiplier">-1.0</param>

File: ur5/mycobot_description/urdf/ur5_robotiq85_gripper.urdf.xacro (robot description, xacro)
@@ -10,5 +10,5 @@
       <geometry>
         <!-- <mesh filename="package://mycobot_gripper_description/meshes/robotiq_85_coupler.stl" /> -->
-        <mesh filename="package://mycobot_gripper_description/meshes/campus02_coupler.stl" />
+        <mesh filename="package://mycobot_gripper_description/meshes/campus02_coupler.dae" />
       </geometry>
       <material name="flat_black"/>
@@ -29,5 +29,5 @@
   <joint name="robotiq_coupler_joint" type="fixed">
     <!-- <origin xyz="0 0 0.004" rpy="0 0 ${-pi/2.0}" /> -->
-    <origin xyz="0 0 -0.01" rpy="0 ${-pi/2.0} ${pi/2.0}" />
+    <origin xyz="0 0 -0.01" rpy="0 ${-pi/2.0} ${-pi/2.0}" />
     <parent link="tool0"/>
     <child link="robotiq_coupler"/>
@@ -48,5 +48,5 @@
   <xacro:robotiq_85_gripper prefix="" parent="robotiq_coupler" >
     <!-- <origin xyz="0 0 0.004" rpy="0 ${-pi/2} ${pi}"/> -->
-    <origin xyz="0.115 0 0" rpy="0 0 0"/>
+    <origin xyz="0.115 0 0" rpy="${pi/2.0} 0 0"/>
   </xacro:robotiq_85_gripper>
   <!-- Gazebo FT sensor plugin -->

File: ur5/mycobot_moveit/srdf/ur_gripper_macro.srdf.xacro (robot description, xacro)
@@ -17,13 +17,13 @@
         <joint name="robotiq_85_left_knuckle_joint" />
     </group>
-    <end_effector name="gripper" parent_link="ee_link" group="gripper" />
+    <end_effector name="eef_gripper" parent_link="ee_link" group="gripper" />
     <!--GROUP STATES - Purpose - Define a named state for a particular group, in terms of joint values. This is useful to define states like 'folded arms' -->
     <group_state name="home" group="arm_controller">
-      <joint name="elbow_joint" value="-1.57" />
+      <joint name="shoulder_pan_joint" value="0.0" />
       <joint name="shoulder_lift_joint" value="-1.57" />
-      <joint name="shoulder_pan_joint" value="1.57" />
-      <joint name="wrist_1_joint" value="0" />
-      <joint name="wrist_2_joint" value="0" />
-      <joint name="wrist_3_joint" value="0" />
+      <joint name="elbow_joint" value="0.0" />
+      <joint name="wrist_1_joint" value="-1.57" />
+      <joint name="wrist_2_joint" value="0.0" />
+      <joint name="wrist_3_joint" value="0.0" />
     </group_state>
     <group_state name="up" group="arm_controller">
@@ -44,8 +44,8 @@
     </group_state>
     <group_state name="closed" group="gripper">
-        <joint name="robotiq_85_left_knuckle_joint" value="0.62" />
+        <joint name="robotiq_85_left_knuckle_joint" value="0.66" />
     </group_state>
     <group_state name="open" group="gripper">
-        <joint name="robotiq_85_left_knuckle_joint" value="0.2" />
+        <joint name="robotiq_85_left_knuckle_joint" value="0.4" />
     </group_state>
     <!-- <group_state name="home" group="arm_gripper_controller">
