Commit message: deleted:    plugins/README.md 	deleted:    plugins/moveit_task_constructor 	deleted:    plugins/rviz2-panel/CMakeLists.txt 	deleted:    plugins/rviz2-panel/LICENSE 	deleted:    plugins/rviz2-panel/include/rviz2-panel/rviz2_panel.hpp 	deleted:    plugins/rviz2-panel/launch/start.launch.py 	deleted:    plugins/rviz2-panel/package.xml 	deleted:    plugins/rviz2-panel/resource/push_button.ui 	deleted:    plugins/rviz2-panel/rviz2/config.rviz 	deleted:    plugins/rviz2-panel/rviz2_plugin.xml 	deleted:    plugins/rviz2-panel/src/rviz2_panel.cpp 	renamed:    ur5/mycobot_mtc/LICENSE -> ur5/mycobot_conveyor_belt/LICENSE 	new file:   ur5/mycobot_conveyor_belt/mycobot_conveyor_belt/__init__.py 	new file:   ur5/mycobot_conveyor_belt/mycobot_conveyor_belt/__pycache__/__init__.cpython-312.pyc 	new file:   ur5/mycobot_conveyor_belt/mycobot_conveyor_belt/__pycache__/conveyor_belt.cpython-312.pyc 	new file:   ur5/mycobot_conveyor_belt/mycobot_conveyor_belt/conveyor_belt.py 	new file:   ur5/mycobot_conveyor_belt/package.xml 	new file:   ur5/mycobot_conveyor_belt/resource/mycobot_conveyor_belt 	new file:   ur5/mycobot_conveyor_belt/setup.cfg 	new file:   ur5/mycobot_conveyor_belt/setup.py 	new file:   ur5/mycobot_conveyor_belt/test/test_copyright.py 	new file:   ur5/mycobot_conveyor_belt/test/test_flake8.py 	new file:   ur5/mycobot_conveyor_belt/test/test_pep257.py 	new file:   ur5/mycobot_description/meshes/conveyor_belt/collision/conveyor_belt.stl 	new file:   ur5/mycobot_description/meshes/conveyor_belt/visual/conveyor_belt.dae 	modified:   ur5/mycobot_description/urdf/ur.urdf.xacro 	new file:   ur5/mycobot_description/urdf/workspace/conveyor_belt.urdf.xacro 	modified:   ur5/mycobot_description/urdf/workspace/workspace.urdf.xacro 	modified:   ur5/mycobot_gazebo/config/ros_gz_bridge.yaml 	modified:   ur5/mycobot_gazebo/models/camera/camera.sdf 	deleted:    ur5/mycobot_gazebo/models/storage/collision/storage.stl 	deleted:    ur5/mycobot_gazebo/models/storage/model.config 	deleted:    ur5/mycobot_gazebo/models/storage/storage.sdf 	deleted:    ur5/mycobot_gazebo/models/storage/visual/storage.dae 	modified:   ur5/mycobot_gazebo/worlds/gazebo.world.sdf 	new file:   ur5/mycobot_interface/LICENSE 	new file:   ur5/mycobot_interface/human_machine_interface.ui 	new file:   ur5/mycobot_interface/mycobot_interface/__init__.py 	new file:   ur5/mycobot_interface/mycobot_interface/__pycache__/__init__.cpython-312.pyc 	new file:   ur5/mycobot_interface/mycobot_interface/__pycache__/hmi.cpython-312.pyc 	new file:   ur5/mycobot_interface/mycobot_interface/__pycache__/resources_rc.cpython-312.pyc 	new file:   ur5/mycobot_interface/mycobot_interface/__pycache__/workpiece.cpython-312.pyc 	new file:   ur5/mycobot_interface/mycobot_interface/hmi.py 	new file:   ur5/mycobot_interface/mycobot_interface/resources_rc.py 	new file:   ur5/mycobot_interface/mycobot_interface/workpiece.py 	new file:   ur5/mycobot_interface/package.xml 	new file:   ur5/mycobot_interface/resource/images/icons/icon_restart.png 	new file:   ur5/mycobot_interface/resource/images/icons/icon_run.png 	new file:   ur5/mycobot_interface/resource/images/logos/camera.png 	new file:   ur5/mycobot_interface/resource/images/logos/conveyor-belt.png 	new file:   ur5/mycobot_interface/resource/images/logos/robotic-arm.png 	new file:   ur5/mycobot_interface/resource/mycobot_interface 	new file:   ur5/mycobot_interface/resource/resources.qrc 	new file:   ur5/mycobot_interface/setup.cfg 	new file:   ur5/mycobot_interface/setup.py 	new file:   ur5/mycobot_interface/test/test_copyright.py 	new file:   ur5/mycobot_interface/test/test_flake8.py 	new file:   ur5/mycobot_interface/test/test_pep257.py 	deleted:    ur5/mycobot_mtc/CMakeLists.txt 	deleted:    ur5/mycobot_mtc/include/mycobot_mtc/mtc_task_common.hpp 	deleted:    ur5/mycobot_mtc/include/mycobot_mtc/mtc_task_node.hpp 	deleted:    ur5/mycobot_mtc/package.xml 	deleted:    ur5/mycobot_mtc/src/mtc_task_callbacks.cpp 	deleted:    ur5/mycobot_mtc/src/mtc_task_creation.cpp 	deleted:    ur5/mycobot_mtc/src/mtc_task_execute.cpp 	deleted:    ur5/mycobot_mtc/src/mtc_task_main.cpp 	deleted:    ur5/mycobot_mtc/src/mtc_task_scene.cpp 	modified:   ur5/mycobot_opencv/mycobot_opencv/__pycache__/__init__.cpython-312.pyc 	modified:   ur5/mycobot_opencv/mycobot_opencv/__pycache__/img_pubsub.cpython-312.pyc 	modified:   ur5/mycobot_opencv/mycobot_opencv/img_pubsub.py 	modified:   ur5/mycobot_opencv/package.xml 	new file:   ur5/mycobot_robot/LICENSE 	new file:   ur5/mycobot_robot/mycobot_robot/__init__.py 	new file:   ur5/mycobot_robot/mycobot_robot/robot_movement.py 	new file:   ur5/mycobot_robot/package.xml 	new file:   ur5/mycobot_robot/resource/mycobot_robot 	new file:   ur5/mycobot_robot/setup.cfg 	new file:   ur5/mycobot_robot/setup.py 	new file:   ur5/mycobot_robot/test/test_copyright.py 	new file:   ur5/mycobot_robot/test/test_flake8.py 	new file:   ur5/mycobot_robot/test/test_pep257.py 	modified:   ur5/mycobot_ros2/CMakeLists.txt 	renamed:    ur5/mycobot_mtc/launch/run.launch.py -> ur5/mycobot_ros2/launch/run.launch.py 	modified:   ur5/mycobot_ros2/package.xml 	renamed:    ur5/mycobot_mtc/rviz/mtc_rviz.rviz -> ur5/mycobot_ros2/rviz/rviz.rviz

File: ur5/mycobot_description/urdf/ur.urdf.xacro (robot description, xacro)
@@ -5,4 +5,6 @@
     <!-- import main macro -->
     <xacro:include filename="$(find mycobot_description)/urdf/ur_macro.xacro"/>
+    <xacro:include filename="$(find mycobot_description)/urdf/workspace/workspace.urdf.xacro" />
+    <xacro:include filename="$(find mycobot_description)/urdf/workspace/conveyor_belt.urdf.xacro" />
     <xacro:arg name="ur_type" default="ur5"/>
     <!-- parameters -->
@@ -44,8 +46,12 @@
     <!-- create link fixed to the "world" -->
     <link name="world" />
-    <xacro:include filename="$(find mycobot_description)/urdf/workspace/workspace.urdf.xacro" />
+    <!-- Robot fixed workspace -->
     <xacro:workspace parent="world">
       <origin xyz="0 0 0" rpy="0 0 0"/>
     </xacro:workspace>
+    <!-- Conveyor belt -->
+    <xacro:conveyor_belt parent="world">
+      <origin xyz="0.8 0.5 0" rpy="0 0 ${pi/2}"/>
+    </xacro:conveyor_belt>
     <!-- arm -->
     <xacro:ur_robot
@@ -95,4 +101,9 @@
           </ros>
         </plugin>
+        <!-- Conveyor Belt Plugin -->
+        <plugin filename="gz-sim-track-controller-system" name="gz::sim::systems::TrackController">
+            <link>conveyor_surface_link</link>
+            <odometry_publish_frequency>1</odometry_publish_frequency>
+        </plugin>
       </gazebo>
     </xacro:if>

File: ur5/mycobot_description/urdf/workspace/workspace.urdf.xacro (robot description, xacro)
@@ -2,4 +2,5 @@
 <robot xmlns:xacro="http://wiki.ros.org/xacro" name="workspace">
     <xacro:macro name="workspace" params="parent *origin_block">
+        <!-- ======================= TABLE ======================= -->
         <link name="table">
             <visual>
@@ -24,4 +25,5 @@
             <origin xyz="-0.235 -0.235 0" rpy="0 0 ${pi/2}"/>
         </joint>
+        <!-- =================== START STORAGE =================== -->
         <link name="start_storage">
             <visual>
@@ -46,27 +48,4 @@
             <origin xyz="-0.07 -0.385 0.9" rpy="0 0 0"/>
         </joint>
-        <!-- Test obstacle -->
-        <!-- <link name="obstacle">
-            <inertial>
-                <mass value="10.0" />
-                <origin xyz="0 0 0" rpy="0 0 0"/>
-                <inertia ixx="1.0" ixy="0.0" ixz="0.0" iyy="1.0" iyz="0.0" izz="1.0" />
-            </inertial>
-            <visual>
-                <geometry>
-                    <box size="0.2 0.2 0.2" />
-                </geometry>
-            </visual>
-            <collision>
-                <geometry>
-                    <box size="0.02 0.02 0.02" />
-                </geometry>
-            </collision>
-        </link>
-        <joint name="${parent}_obstacle" type="fixed">
-            <parent link="${parent}"/>
-            <child link="obstacle"/>
-            <origin xyz="-0.2 0 1.09" rpy="0 0 0"/>
-        </joint> -->
     </xacro:macro>
 </robot>
