Commit message: modified:   ur5/mycobot_description/urdf/workspace/conveyor_belt.urdf.xacro 	modified:   ur5/mycobot_gazebo/config/ros_gz_bridge.yaml 	modified:   ur5/mycobot_gazebo/models/camera/camera.sdf 	modified:   ur5/mycobot_gazebo/worlds/gazebo.world.sdf 	modified:   ur5/mycobot_interface/human_machine_interface.ui 	modified:   ur5/mycobot_interface/mycobot_interface/__pycache__/hmi.cpython-312.pyc 	modified:   ur5/mycobot_interface/mycobot_interface/__pycache__/workpiece.cpython-312.pyc 	modified:   ur5/mycobot_interface/mycobot_interface/hmi.py 	modified:   ur5/mycobot_interface/mycobot_interface/workpiece.py 	modified:   ur5/mycobot_moveit/config/ros2_controllers.yaml 	modified:   ur5/mycobot_opencv/mycobot_opencv/__pycache__/img_pubsub.cpython-312.pyc 	modified:   ur5/mycobot_opencv/mycobot_opencv/img_pubsub.py 	new file:   ur5/mycobot_robot/mycobot_robot/__pycache__/__init__.cpython-312.pyc 	new file:   ur5/mycobot_robot/mycobot_robot/__pycache__/robot_movement.cpython-312.pyc 	new file:   ur5/mycobot_robot/mycobot_robot/__pycache__/trajectory.cpython-312.pyc 	modified:   ur5/mycobot_robot/mycobot_robot/robot_movement.py 	new file:   ur5/mycobot_robot/mycobot_robot/trajectory.py 	modified:   ur5/mycobot_ros2/launch/run.launch.py

File: ur5/mycobot_description/urdf/workspace/conveyor_belt.urdf.xacro (robot description, xacro)
@@ -61,5 +61,5 @@
             <origin xyz="0 0 0.741" rpy="0 0 ${pi/2}"/>
             <axis xyz="1 0 0"/>
-            <limit lower="0.0" upper="0.01" effort="100" velocity="1.0"/>
+            <limit lower="0.0" upper="0.05" effort="100" velocity="1.0"/>
         </joint>
     </xacro:macro>
