Commit message: modified:   ur5/mycobot_description/urdf/workspace/workspace.urdf.xacro 	modified:   ur5/mycobot_gazebo/models/workpiece/collision/workpiece.stl 	new file:   ur5/mycobot_gazebo/models/workpiece/model.config 	deleted:    ur5/mycobot_gazebo/models/workpiece/visual/RobotiQ-2F-85-Gripper-Open.tool 	modified:   ur5/mycobot_gazebo/models/workpiece/visual/workpiece.dae 	new file:   ur5/mycobot_gazebo/models/workpiece/workpiece.sdf 	modified:   ur5/mycobot_gazebo/worlds/gazebo.world.sdf 	modified:   ur5/mycobot_gripper_description/urdf/robotiq_85_gripper.urdf.xacro 	modified:   ur5/mycobot_mtc/launch/run.launch.py 	modified:   ur5/mycobot_mtc/src/mtc_node.cpp

File: ur5/mycobot_description/urdf/workspace/workspace.urdf.xacro (robot description, xacro)
@@ -46,4 +46,27 @@
             <origin xyz="-0.07 -0.385 0.9" rpy="0 0 0"/>
         </joint>
+        <!-- Test obstacle -->
+        <!-- <link name="obstacle">
+            <inertial>
+                <mass value="10.0" />
+                <origin xyz="0 0 0" rpy="0 0 0"/>
+                <inertia ixx="1.0" ixy="0.0" ixz="0.0" iyy="1.0" iyz="0.0" izz="1.0" />
+            </inertial>
+            <visual>
+                <geometry>
+                    <box size="0.2 0.2 0.2" />
+                </geometry>
+            </visual>
+            <collision>
+                <geometry>
+                    <box size="0.02 0.02 0.02" />
+                </geometry>
+            </collision>
+        </link>
+        <joint name="${parent}_obstacle" type="fixed">
+            <parent link="${parent}"/>
+            <child link="obstacle"/>
+            <origin xyz="-0.2 0 1.09" rpy="0 0 0"/>
+        </joint> -->
     </xacro:macro>
 </robot>

File: ur5/mycobot_gripper_description/urdf/robotiq_85_gripper.urdf.xacro (robot description, xacro)
@@ -238,13 +238,13 @@
     <!-- Improve grasping physics -->
     <gazebo reference="${prefix}robotiq_85_left_finger_tip_link">
-      <kp>1000000.0</kp>
-      <kd>1.0</kd>
-      <mu1>1.0</mu1>
-      <mu2>1.0</mu2>
+      <kp>10000000.0</kp>
+      <kd>10.0</kd>
+      <mu1>5.0</mu1>
+      <mu2>5.0</mu2>
       <minDepth>0.001</minDepth>
     </gazebo>
     <gazebo reference="${prefix}robotiq_85_right_finger_tip_link">
-      <kp>1000000.0</kp>
-      <kd>1.0</kd>
+      <kp>10000000.0</kp>
+      <kd>10.0</kd>
       <mu1>1.0</mu1>
       <mu2>1.0</mu2>

Commit message: new file:   plugins/moveit_task_constructor modified:   ur5/mycobot_description/urdf/workspace/workspace.urdf.xacro modified:   ur5/mycobot_interface/mycobot_interface/__pycache__/hmi.cpython-312.pyc modified:   ur5/mycobot_interface/mycobot_interface/hmi.py new file:   ur5/mycobot_mtc/CMakeLists.txt renamed:    ur5/mycobot_robot/LICENSE -> ur5/mycobot_mtc/LICENSE new file:   ur5/mycobot_mtc/include/mycobot_mtc/mtc_task_common.hpp new file:   ur5/mycobot_mtc/include/mycobot_mtc/mtc_task_node.hpp new file:   ur5/mycobot_mtc/package.xml new file:   ur5/mycobot_mtc/src/mtc_task_callbacks.cpp new file:   ur5/mycobot_mtc/src/mtc_task_creation.cpp new file:   ur5/mycobot_mtc/src/mtc_task_execute.cpp new file:   ur5/mycobot_mtc/src/mtc_task_main.cpp new file:   ur5/mycobot_mtc/src/mtc_task_spawn_workpiece.cpp modified:   ur5/mycobot_opencv/mycobot_opencv/__pycache__/img_pubsub.cpython-312.pyc modified:   ur5/mycobot_opencv/mycobot_opencv/img_pubsub.py deleted:    ur5/mycobot_robot/mycobot_robot/__init__.py deleted:    ur5/mycobot_robot/mycobot_robot/__pycache__/__init__.cpython-312.pyc deleted:    ur5/mycobot_robot/mycobot_robot/__pycache__/robot_movement.cpython-312.pyc deleted:    ur5/mycobot_robot/mycobot_robot/__pycache__/trajectory.cpython-312.pyc deleted:    ur5/mycobot_robot/mycobot_robot/robot_movement.py deleted:    ur5/mycobot_robot/mycobot_robot/trajectory.py deleted:    ur5/mycobot_robot/package.xml deleted:    ur5/mycobot_robot/resource/mycobot_robot deleted:    ur5/mycobot_robot/setup.cfg deleted:    ur5/mycobot_robot/setup.py deleted:    ur5/mycobot_robot/test/test_copyright.py deleted:    ur5/mycobot_robot/test/test_flake8.py deleted:    ur5/mycobot_robot/test/test_pep257.py modified:   ur5/mycobot_ros2/launch/run.launch.py modified:   ur5/mycobot_ros2/package.xml modified:   ur5/mycobot_ros2/rviz/rviz.rviz

File: ur5/mycobot_description/urdf/workspace/workspace.urdf.xacro (robot description, xacro)
@@ -26,5 +26,5 @@
         </joint>
         <!-- =================== START STORAGE =================== -->
-        <link name="start_storage">
+        <link name="target_storage">
             <visual>
                 <geometry>
@@ -45,5 +45,5 @@
         <joint name="${parent}_to_start-storage_joint" type="fixed">
             <parent link="${parent}"/>
-            <child link="start_storage"/>
+            <child link="target_storage"/>
             <origin xyz="-0.07 -0.385 0.9" rpy="0 0 0"/>
         </joint>
